File: Hardware/Hotplate/PinHeaderOutputs.kicad_sch (KiCad schematic)
At the start: 4 parts, among them J1 Conn_01x04_Pin, J2 Conn_01x04_Pin, J3 I2C2, J9 SPI3

Commit message: V2
Parts:
- added J10: 5V, Connector_PinHeader_2.54mm:PinHeader_1x02_P2.54mm_Vertical, symbol Connector:Conn_01x02_Pin
- added J4: VCC, Connector_Wire:SolderWire-1.5sqmm_1x01_D1.7mm_OD3mm, symbol Connector:Conn_01x01_Pin
- added J5: GND, Connector_Wire:SolderWire-1.5sqmm_1x01_D1.7mm_OD3mm, symbol Connector:Conn_01x01_Pin
Connections:
- net GND: now also J10.1 (Pin_1), J5.1 (Pin_1)
- new net +5V: J10.2 (Pin_2)
- new net VCC: J4.1 (Pin_1)

Commit message: made it pretty (#8)
Co-authored-by: nexophoenixe <jan.gradwohl2005@mail.com>
Parts:
- renumbered J4 to J501, J5 to J502, J1 to J503, J2 to J504, J3 to J505, J9 to J506, J10 to J507
Other:
- note added: "I2C2"
- note added: "Main Powersupply"
- note added: "SPI3"
- note added: "STM32 Prog."
- note added: "USART1"
- note added: "USB VBUS"
- moved on the sheet: J501, J502, J503, J504, J505, J506, J507
