File: Hardware/Hotplate/Power.kicad_sch (KiCad schematic)
At the start: 7 parts, among them IC1 TL783CKCSE3

Commit message: made it pretty (#8)
Co-authored-by: nexophoenixe <jan.gradwohl2005@mail.com>
Parts:
- renumbered C8 to C301, C7 to C302, D4 to D301, IC1 to IC301, R7 to R301, R6 to R302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
Other:
- note added: "3.3V Indicator"
- note added: "LDO 48V-3.3V"
- moved on the sheet: C301, C302, D301, IC301, R301, R302, R303
