File: Hardware/Hotplate/TempSens.kicad_sch (KiCad schematic)
At the start: 6 parts, among them J6 PA1, J7 PA0

Commit message: Updated Kicad 8 to 9
Changed lines of the file:
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@@
 (kicad_sch
-	(version 20231120)
+	(version 20250114)
 	(generator "eeschema")
-	(generator_version "8.0")
+	(generator_version "9.0")
 	(paper "A4")
 	(junction

Commit message: made it pretty (#8)
Co-authored-by: nexophoenixe <jan.gradwohl2005@mail.com>
Parts:
- renumbered C5 to C401, C4 to C402, J7 to J401, J6 to J402, R5 to R401, R4 to R402
Other:
- note added: "Temp Sens PA0"
- note added: "Temp Sens PA1"
- moved on the sheet: C401, C402, J401, J402, R401, R402
