File: Hardware/Hotplate/Hotplate.kicad_pcb (KiCad board)
At the start: 2 copper layers, 114.2 x 118.4 mm, 54 parts, among them IC1 TL783CKCSE3, IC2 FT231XQ-T, J1 Conn_01x04_Pin, J2 Conn_01x04_Pin, J3 I2C2, J4 Conn_01x01_Pin, J5 Conn_01x01_Pin, J6 PA1, J7 PA0, J8 GSB1C41110SSHR, J9 SPI3, Q2 Q_NMOS_GDS, SW1 SW_Push, SW2 SW_Push, SW3 SW_Push, SW4 SW_Push, U1 STM32F301K6Tx

Commit message: V2
Parts:
- removed Q2: Q_NMOS_GDS, Package_TO_SOT_SMD:TO-252-2
- removed R2: 1k, Resistor_SMD:R_0805_2012Metric
- removed R3: 100k, Resistor_SMD:R_0805_2012Metric
- added C11: 1uF, Capacitor_SMD:C_0603_1608Metric, F.Cu at (148.0, 55.9)
- added D7: D_Schottky, Diode_THT:D_DO-15_P10.16mm_Horizontal, F.Cu at (143.3, 54.2)
- added IC4: FT231XS-U, SamacSys_Parts:SOP64P599X175-20N, F.Cu at (142.7, 147.4)
- added J10: 5V, Connector_PinHeader_2.54mm:PinHeader_1x02_P2.54mm_Vertical, F.Cu at (155.4, 133.1)
- added Q1: BSC146N10LS5ATMA1, SamacSys_Parts:BSC146N10LS5ATMA1, F.Cu at (151.0, 66.3)
- added R11: 270, Resistor_SMD:R_0603_1608Metric_Pad0.98x0.95mm_HandSolder, F.Cu at (150.2, 60.1)
- C1, C2: value C -> 100nF
- C3: value C -> 10nF
- C6: moved to F.Cu
- IC2: value FT231XQ-T -> MCP1402T-E_OT; footprint SamacSys_Parts:QFN50P400X400X80-21N -> SamacSys_Parts:SOT95P270X145-5N
- J4: value Conn_01x01_Pin -> VCC
- J5: value Conn_01x01_Pin -> GND
- moved IC2 88.6 mm to (147.6, 59.0), turned to -90 degrees
- moved R9 12.5 mm to (153.4, 152.4)
- moved D1 12.4 mm to (155.0, 152.4), turned to 90 degrees
- moved H1 10.4 mm to (36.0, 51.0)
- moved H2 10.1 mm to (36.2, 161.5)
- moved H4 4.88 mm to (132.4, 161.8)
- moved C9 4.55 mm to (150.8, 147.5)
- moved C6 2.28 mm to (153.8, 109.8), turned to 180 degrees
- moved C10 1.95 mm to (150.8, 149.3)
- moved C12 0.29 mm to (149.9, 155.5)
- moved C13 0.29 mm to (146.3, 155.5)
- moved R12 0.29 mm to (147.3, 152.6)
- moved R13 0.29 mm to (149.0, 152.6)
- moved J5 0.09 mm to (155.0, 59.2)
- moved J4 0.06 mm to (155.0, 54.1)
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Connections:
- IC2 pad 1: USART1_TX -> GND
- IC2 pad 2: unconnected-(IC2-RI#-Pad2) -> +5V
- IC2 pad 3: GND -> PA2 | TIM2_CH3
- IC2 pad 4: unconnected-(IC2-DSR#-Pad4) -> GND
- IC2 pad 5: unconnected-(IC2-DCD#-Pad5) -> Net-(IC2-OUT)
- NT1 pad 1: Net-(Q2-D) -> Drain
- R12 pad 2: Net-(IC2-USBDP) -> USBDP
- R13 pad 2: Net-(IC2-USBDM) -> USBDM
- R15 pad 1: Net-(IC2-CBUS1) -> CBUS1
- R16 pad 1: Net-(IC2-CBUS0) -> CBUS0
- U1 pad 8: Net-(U1-PA2) -> PA2 | TIM2_CH3
Routing:
- net +5V: track 29.9 -> 137.7 mm, vias 0 -> 1
- net PA2 | TIM2_CH3: track 0.00 -> 52.5 mm, vias 0 -> 2
- net Net-(U1-PA2): track 39.4 -> 0.00 mm, vias 2 -> 0
- net VCC: track 7269.9 -> 7292.2 mm
- net Drain: track 0.00 -> 12.2 mm
- net CBUS1: track 0.00 -> 10.3 mm
- net Net-(Q2-D): track 8.73 -> 0.00 mm
- net CBUS0: track 0.00 -> 8.33 mm
- net Net-(IC2-CBUS1): track 7.24 -> 0.00 mm
- net USART1_TX: track 48.1 -> 41.3 mm, vias 2 -> 1
- net Net-(Q2-G): track 5.46 -> 0.00 mm
- net USBDM: track 0.00 -> 5.26 mm
- net Net-(IC2-CBUS0): track 4.85 -> 0.00 mm
- net VCCIO: track 16.7 -> 13.0 mm
- net USBDP: track 0.00 -> 2.98 mm
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- added copper zone on F.Cu, net Drain
Other:
- board size 114.2 x 118.4 mm -> 125.3 x 118.4 mm

Commit message: made it pretty (#8)
Co-authored-by: nexophoenixe <jan.gradwohl2005@mail.com>
Parts:
- renumbered C2 to C101, C1 to C102, C6 to C103, C3 to C104, C11 to C105, C12 to C201, C13 to C202, C10 to C203, C9 to C204, C8 to C301, C7 to C302, C5 to C401, C4 to C402, D5 to D101, D6 to D102, D7 to D103, D1 to D201, D2 to D202, D3 to D203, D4 to D301, H1 to H101, H2 to H102, H3 to H103, H4 to H104, IC2 to IC101, IC4 to IC201, IC1 to IC301, J8 to J201, J7 to J401, J6 to J402, J4 to J501, J5 to J502, J1 to J503, J2 to J504, J3 to J505, J9 to J506, J10 to J507, NT1 to NT101, Q1 to Q101, R17 to R101, R8 to R102, R11 to R103, R9 to R201, R15 to R202, R16 to R203, R12 to R204, R13 to R205, R7 to R301, R6 to R302, R1 to R303, R5 to R401, R4 to R402, SW4 to SW101, SW3 to SW102, SW2 to SW103, SW1 to SW104, U1 to U101

Commit message: Debug (#15)
* fixed:PID

* fixed:PID

* fixed:dyingFETs
Parts:
- R103: value 270 -> 0
Changed lines of the file:
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@@
 			)
 		)
-		(property "Value" "270"
+		(property "Value" "0"
 			(at 0 -1.1 90)
 			(layer "F.SilkS")
@@
 			(at 0 0 0)
 			(layer "F.SilkS")
-			(hide yes)
 			(effects
 				(font
@@
 			(keep_text_aligned yes)
 		)
-		(gr_text "110.0000 mm"
+		(gr_text "110,0000 mm"
 			(at 23.2 106.35 90)
 			(layer "User.4")
@@
 			(keep_text_aligned yes)
 		)
-		(gr_text "91.0000 mm"
+		(gr_text "91,0000 mm"
 			(at 92.85 17.2 0)
 			(layer "User.4")
@@
 			(keep_text_aligned yes)
 		)
-		(gr_text "110.0000 mm"
+		(gr_text "110,0000 mm"
 			(at 102.35 172.199999 0)
 			(layer "User.4")
@@
 			(keep_text_aligned yes)
 		)
-		(gr_text "2.2000 mm"
+		(gr_text "2,2000 mm"
 			(at 40.443286 160.65 0)
 			(layer "User.4")
